File: kicad/schematic-final/schematic-final.kicad_sch (KiCad schematic)
At the start: 12 parts

Commit message: (#12) Removed LCD from schematic and README
Parts:
- removed J?: 1602_I2C, symbol Treadmill:1602_I2C
